File: pcb/digit-module/digit-module.kicad_pcb (KiCad board)
At the start: 2 copper layers, 20 parts, among them J1 Conn_01x09_Male, J2 STM32_SWD, Q1 PZT2222A, Q2 PZT2222A, U1 STM32F030F4Px

Commit message: Digit display enclosure and PCB draft routing
However, still need to verify that everything fits together before
milling/printing

Exact transistor/LED values also need to be confirmed...
Connections:
- U1 pad 14: Net-(U1-Pad14) -> Net-(J1-Pad5)
- U1 pad 17: Net-(U1-Pad17) -> Net-(J1-Pad4)
- U1 pad 18: Net-(U1-Pad18) -> Net-(J1-Pad3)
Routing:
- net Net-(J1-Pad3): track 0.00 -> 60.8 mm, vias 0 -> 1
- net Net-(J1-Pad4): track 0.00 -> 60.6 mm, vias 0 -> 1
- net Net-(J1-Pad5): track 0.00 -> 57.0 mm, vias 0 -> 1
