File: pcb/digit-module/digit-module.sch (KiCad schematic (older format))
At the start: 3 parts, among them Q1 PN2222A, Q2 PN2222A, U1 STM32F030F4Px

Commit message: Digit display enclosure and PCB draft routing
However, still need to verify that everything fits together before
milling/printing

Exact transistor/LED values also need to be confirmed...
Parts:
- added C1, C2, C3: CP, Capacitor_SMD:C_0603_1608Metric, symbol device:CP
- added J1: Conn_01x09_Male, Connector_PinHeader_2.54mm:PinHeader_1x09_P2.54mm_Horizontal, symbol conn:Conn_01x09_Male
- added J2: STM32_SWD, Connector_PinHeader_2.54mm:PinHeader_1x05_P2.54mm_Horizontal, symbol custom:STM32_SWD
- added R1, R2: 100, Resistors_SMD:R_0603, symbol device:R
- Q1, Q2: value PN2222A -> PZT2222A; footprint Package_TO_SOT_THT:TO-92 -> Package_TO_SOT_SMD:SOT-223-3_TabPin2; symbol Transistor_BJT:PN2222A -> Transistor_BJT:PZT2222A
Connections:
- net labels added: VDD, VDDA
- wire segments 27 -> 61
- no-connect marks 0 -> 1
