File: pcb/digit-node-breakout/led_matrix.sch (KiCad schematic (older format))
At the start: 10 parts

Commit message: Renamed digit-module for consistency
Parts:
- D1, D10, D2, D3, D4, D5, D6, D7, D8, D9: footprint LEDs:LED_0603 -> LED_SMD:LED_0603_1608Metric
Changed lines of the file:
@@
 EESchema Schematic File Version 4
-LIBS:digit-module-cache
+LIBS:digit-node-cache
 EELAYER 26 0
 EELAYER END
@@
 F 0 "D1" H 1600 750 50  0000 C CNN
 F 1 "LED_0" H 1600 550 50  0000 C CNN
-F 2 "LEDs:LED_0603" H 1600 650 50  0001 C CNN
+F 2 "LED_SMD:LED_0603_1608Metric" H 1600 650 50  0001 C CNN
 F 3 "" H 1600 650 50  0001 C CNN
 	1    1600 650
@@
 F 0 "D2" H 1600 1050 50  0000 C CNN
 F 1 "LED_1" H 1600 850 50  0000 C CNN
-F 2 "LEDs:LED_0603" H 1600 950 50  0001 C CNN
+F 2 "LED_SMD:LED_0603_1608Metric" H 1600 950 50  0001 C CNN
 F 3 "" H 1600 950 50  0001 C CNN
 	1    1600 950
@@
 F 0 "D3" H 1600 1350 50  0000 C CNN
 F 1 "LED_2" H 1600 1150 50  0000 C CNN
-F 2 "LEDs:LED_0603" H 1600 1250 50  0001 C CNN
+F 2 "LED_SMD:LED_0603_1608Metric" H 1600 1250 50  0001 C CNN
 F 3 "" H 1600 1250 50  0001 C CNN
 	1    1600 1250
@@
 F 0 "D4" H 1600 1650 50  0000 C CNN
 F 1 "LED_3" H 1600 1450 50  0000 C CNN
-F 2 "LEDs:LED_0603" H 1600 1550 50  0001 C CNN
+F 2 "LED_SMD:LED_0603_1608Metric" H 1600 1550 50  0001 C CNN
 F 3 "" H 1600 1550 50  0001 C CNN
 	1    1600 1550
@@
 F 0 "D5" H 1600 1950 50  0000 C CNN
 F 1 "LED_4" H 1600 1750 50  0000 C CNN
-F 2 "LEDs:LED_0603" H 1600 1850 50  0001 C CNN
+F 2 "LED_SMD:LED_0603_1608Metric" H 1600 1850 50  0001 C CNN
 F 3 "" H 1600 1850 50  0001 C CNN
 	1    1600 1850
@@
 F 0 "D6" H 1600 2250 50  0000 C CNN
 F 1 "LED_5" H 1600 2050 50  0000 C CNN
-F 2 "LEDs:LED_0603" H 1600 2150 50  0001 C CNN
+F 2 "LED_SMD:LED_0603_1608Metric" H 1600 2150 50  0001 C CNN
 F 3 "" H 1600 2150 50  0001 C CNN
 	1    1600 2150
@@
 F 0 "D7" H 1600 2550 50  0000 C CNN
 F 1 "LED_6" H 1600 2350 50  0000 C CNN
-F 2 "LEDs:LED_0603" H 1600 2450 50  0001 C CNN
+F 2 "LED_SMD:LED_0603_1608Metric" H 1600 2450 50  0001 C CNN
 F 3 "" H 1600 2450 50  0001 C CNN
 	1    1600 2450
@@
 F 0 "D8" H 1600 2850 50  0000 C CNN
 F 1 "LED_7" H 1600 2650 50  0000 C CNN
-F 2 "LEDs:LED_0603" H 1600 2750 50  0001 C CNN
+F 2 "LED_SMD:LED_0603_1608Metric" H 1600 2750 50  0001 C CNN
 F 3 "" H 1600 2750 50  0001 C CNN
 	1    1600 2750
@@
 F 0 "D9" H 1600 3150 50  0000 C CNN
 F 1 "LED_8" H 1600 2950 50  0000 C CNN
-F 2 "LEDs:LED_0603" H 1600 3050 50  0001 C CNN
+F 2 "LED_SMD:LED_0603_1608Metric" H 1600 3050 50  0001 C CNN
 F 3 "" H 1600 3050 50  0001 C CNN
 	1    1600 3050
@@
 F 0 "D10" H 1600 3450 50  0000 C CNN
 F 1 "LED_9" H 1600 3250 50  0000 C CNN
-F 2 "LEDs:LED_0603" H 1600 3350 50  0001 C CNN
+F 2 "LED_SMD:LED_0603_1608Metric" H 1600 3350 50  0001 C CNN
 F 3 "" H 1600 3350 50  0001 C CNN
 	1    1600 3350
