File: pcb/digit-node-breakout/digit-node.sch (KiCad schematic (older format))
At the start: 10 parts, among them J1 Conn_01x09_Male, J2 STM32_SWD, Q1 PZT2222A, Q2 PZT2222A, U1 STM32F030F4Px

Commit message: Renamed digit-module for consistency
Parts:
- R1, R2: footprint Resistors_SMD:R_0603 -> Resistor_SMD:R_0603_1608Metric
- U1: footprint Housings_SSOP:TSSOP-20_4.4x6.5mm_Pitch0.65mm -> Package_SO:TSSOP-20_4.4x6.5mm_P0.65mm
Changed lines of the file:
@@
 EESchema Schematic File Version 4
-LIBS:digit-module-cache
+LIBS:digit-node-cache
 EELAYER 26 0
 EELAYER END
@@
 F 0 "U1" H 3400 2164 50  0000 C CNN
 F 1 "STM32F030F4Px" H 3400 2073 50  0000 C CNN
-F 2 "Housings_SSOP:TSSOP-20_4.4x6.5mm_Pitch0.65mm" H 5000 4025 50  0001 R TNN
+F 2 "Package_SO:TSSOP-20_4.4x6.5mm_P0.65mm" H 5000 4025 50  0001 R TNN
 F 3 "http://www.st.com/st-web-ui/static/active/en/resource/technical/document/datasheet/DM00088500.pdf" H 3400 3150 50  0001 C CNN
 	1    3400 3150
@@
 F 0 "R1" H 7470 2996 50  0000 L CNN
 F 1 "100" H 7470 2905 50  0000 L CNN
-F 2 "Resistors_SMD:R_0603" V 7330 2950 50  0001 C CNN
+F 2 "Resistor_SMD:R_0603_1608Metric" V 7330 2950 50  0001 C CNN
 F 3 "" H 7400 2950 50  0001 C CNN
 	1    7400 2950
@@
 F 0 "R2" H 7720 2996 50  0000 L CNN
 F 1 "100" H 7720 2905 50  0000 L CNN
-F 2 "Resistors_SMD:R_0603" V 7580 2950 50  0001 C CNN
+F 2 "Resistor_SMD:R_0603_1608Metric" V 7580 2950 50  0001 C CNN
 F 3 "" H 7650 2950 50  0001 C CNN
 	1    7650 2950

Commit message: More digit PCB cleanup
Parts:
- U1: symbol stm32:STM32F030F4Px -> MCU_ST_STM32F0:STM32F030F4Px
Connections:
- wire segments 61 -> 64
Changed lines of the file:
@@
 $EndSheet
 $Comp
-L stm32:STM32F030F4Px U1
+L MCU_ST_STM32F0:STM32F030F4Px U1
 U 1 1 5AE88544
-P 3400 3150
-F 0 "U1" H 3400 2164 50  0000 C CNN
-F 1 "STM32F030F4Px" H 3400 2073 50  0000 C CNN
-F 2 "Package_SO:TSSOP-20_4.4x6.5mm_P0.65mm" H 5000 4025 50  0001 R TNN
-F 3 "http://www.st.com/st-web-ui/static/active/en/resource/technical/document/datasheet/DM00088500.pdf" H 3400 3150 50  0001 C CNN
-	1    3400 3150
+P 3400 3050
+F 0 "U1" H 3400 2064 50  0000 C CNN
+F 1 "STM32F030F4Px" H 3400 1973 50  0000 C CNN
+F 2 "Package_SO:TSSOP-20_4.4x6.5mm_P0.65mm" H 5000 3925 50  0001 R TNN
+F 3 "http://www.st.com/st-web-ui/static/active/en/resource/technical/document/datasheet/DM00088500.pdf" H 3400 3050 50  0001 C CNN
+	1    3400 3050
 	1    0    0    -1
 $EndComp
@@
 Connection ~ 7400 3900
 Wire Wire Line
-	5750 3350 7100 3350
-Wire Wire Line
-	5700 3700 7350 3700
+	5800 3350 7100 3350
+Wire Wire Line
+	5900 3700 7350 3700
 Wire Wire Line
 	5800 2550 6350 2550
@@
 $EndComp
 Wire Wire Line
-	1250 2550 1700 2550
-Wire Wire Line
-	5100 3650 5100 4300
-Wire Wire Line
-	5100 4300 1600 4300
-Wire Wire Line
-	5100 3550 5150 3550
-Wire Wire Line
-	5150 3550 5150 4350
+	4000 3650 4000 4200
+Wire Wire Line
+	4000 4200 2600 4200
+Wire Wire Line
+	4100 3550 4100 4300
 $Comp
 L power:GND #PWR08
 U 1 1 5AE8E4D7
-P 3400 4050
-F 0 "#PWR08" H 3400 3800 50  0001 C CNN
-F 1 "GND" H 3405 3877 50  0000 C CNN
-F 2 "" H 3400 4050 50  0001 C CNN
-F 3 "" H 3400 4050 50  0001 C CNN
-	1    3400 4050
-	1    0    0    -1
+P 3400 3850
+F 0 "#PWR08" H 3400 3600 50  0001 C CNN
+F 1 "GND" H 3405 3677 50  0000 C CNN
+F 2 "" H 3400 3850 50  0001 C CNN
+F 3 "" H 3400 3850 50  0001 C CNN
+	1    3400 3850
+	0    -1   -1   0
 $EndComp
 $Comp
 L device:CP C2
 U 1 1 5AE8E5A1
-P 3550 2050
-F 0 "C2" V 3805 2050 50  0000 C CNN
-F 1 "CP" V 3714 2050 50  0000 C CNN
-F 2 "Capacitor_SMD:C_0603_1608Metric" H 3588 1900 50  0001 C CNN
-F 3 "" H 3550 2050 50  0001 C CNN
-	1    3550 2050
+P 3650 2050
+F 0 "C2" V 3905 2050 50  0000 C CNN
+F 1 "CP" V 3814 2050 50  0000 C CNN
+F 2 "Capacitor_SMD:C_0603_1608Metric" H 3688 1900 50  0001 C CNN
+F 3 "" H 3650 2050 50  0001 C CNN
+	1    3650 2050
 	0    -1   -1   0
 $EndComp
@@
 L device:CP C3
 U 1 1 5AE8E65E
-P 3850 2050
-F 0 "C3" V 4105 2050 50  0000 C CNN
-F 1 "CP" V 4014 2050 50  0000 C CNN
-F 2 "Capacitor_SMD:C_0603_1608Metric" H 3888 1900 50  0001 C CNN
-F 3 "" H 3850 2050 50  0001 C CNN
-	1    3850 2050
+P 3950 2050
+F 0 "C3" V 4205 2050 50  0000 C CNN
+F 1 "CP" V 4114 2050 50  0000 C CNN
+F 2 "Capacitor_SMD:C_0603_1608Metric" H 3988 1900 50  0001 C CNN
+F 3 "" H 3950 2050 50  0001 C CNN
+	1    3950 2050
 	0    -1   -1   0
 $EndComp
@@
 L device:CP C1
 U 1 1 5AE8E71F
-P 3150 2050
-F 0 "C1" V 2895 2050 50  0000 C CNN
-F 1 "CP" V 2986 2050 50  0000 C CNN
-F 2 "Capacitor_SMD:C_0603_1608Metric" H 3188 1900 50  0001 C CNN
-F 3 "" H 3150 2050 50  0001 C CNN
-	1    3150 2050
-	0    1    1    0
-$EndComp
-Wire Wire Line
-	3300 2150 3300 2050
-Wire Wire Line
-	3400 2050 3400 2150
+P 3250 2050
+F 0 "C1" V 2995 2050 50  0000 C CNN
+F 1 "CP" V 3086 2050 50  0000 C CNN
+F 2 "Capacitor_SMD:C_0603_1608Metric" H 3288 1900 50  0001 C CNN
+F 3 "" H 3250 2050 50  0001 C CNN
+	1    3250 2050
+	0    1    1    0
+$EndComp
 $Comp
 L power:VDD #PWR07
 U 1 1 5AE8FF5E
-P 3250 1850
-F 0 "#PWR07" H 3250 1700 50  0001 C CNN
-F 1 "VDD" H 3267 2023 50  0000 C CNN
-F 2 "" H 3250 1850 50  0001 C CNN
-F 3 "" H 3250 1850 50  0001 C CNN
-	1    3250 1850
+P 3350 1850
+F 0 "#PWR07" H 3350 1700 50  0001 C CNN
+F 1 "VDD" H 3367 2023 50  0000 C CNN
+F 2 "" H 3350 1850 50  0001 C CNN
+F 3 "" H 3350 1850 50  0001 C CNN
+	1    3350 1850
 	1    0    0    -1
 $EndComp
@@
 L power:VDDA #PWR09
 U 1 1 5AE90007
-P 3450 1850
-F 0 "#PWR09" H 3450 1700 50  0001 C CNN
-F 1 "VDDA" H 3467 2023 50  0000 C CNN
-F 2 "" H 3450 1850 50  0001 C CNN
-F 3 "" H 3450 1850 50  0001 C CNN
-	1    3450 1850
+P 3550 1850
+F 0 "#PWR09" H 3550 1700 50  0001 C CNN
+F 1 "VDDA" H 3567 2023 50  0000 C CNN
+F 2 "" H 3550 1850 50  0001 C CNN
+F 3 "" H 3550 1850 50  0001 C CNN
+	1    3550 1850
 	1    0    0    -1
 $EndComp
@@
 	1    0    0    -1
 $EndComp
-Connection ~ 3300 2050
-Wire Wire Line
-	3250 1850 3300 1850
-Wire Wire Line
-	3300 1850 3300 2050
-Wire Wire Line
-	3450 1850 3400 1850
+Connection ~ 3400 2050
+Wire Wire Line
+	3350 1850 3400 1850
 Wire Wire Line
 	3400 1850 3400 2050
-Connection ~ 3400 2050
+Wire Wire Line
+	3550 1850 3500 1850
+Wire Wire Line
+	3500 1850 3500 2050
+Connection ~ 3500 2050
 $Comp
 L power:GND #PWR06
 U 1 1 5AE9CD7D
-P 3000 2050
-F 0 "#PWR06" H 3000 1800 50  0001 C CNN
-F 1 "GND" V 3005 1922 50  0000 R CNN
-F 2 "" H 3000 2050 50  0001 C CNN
-F 3 "" H 3000 2050 50  0001 C CNN
-	1    3000 2050
+P 3100 2050
+F 0 "#PWR06" H 3100 1800 50  0001 C CNN
+F 1 "GND" V 3105 1922 50  0000 R CNN
+F 2 "" H 3100 2050 50  0001 C CNN
+F 3 "" H 3100 2050 50  0001 C CNN
+	1    3100 2050
 	0    1    1    0
 $EndComp
@@
 L power:GND #PWR010
 U 1 1 5AE9CDD1
-P 4000 2050
-F 0 "#PWR010" H 4000 1800 50  0001 C CNN
-F 1 "GND" V 4005 1922 50  0000 R CNN
-F 2 "" H 4000 2050 50  0001 C CNN
-F 3 "" H 4000 2050 50  0001 C CNN
-	1    4000 2050
+P 4100 2050
+F 0 "#PWR010" H 4100 1800 50  0001 C CNN
+F 1 "GND" V 4105 1922 50  0000 R CNN
+F 2 "" H 4100 2050 50  0001 C CNN
+F 3 "" H 4100 2050 50  0001 C CNN
+	1    4100 2050
 	0    -1   -1   0
 $EndComp
@@
 $EndComp
 Wire Wire Line
-	5150 4350 1550 4350
-Wire Wire Line
-	1600 4300 1600 2850
-Wire Wire Line
-	1250 2850 1600 2850
-Wire Wire Line
-	1550 4350 1550 2650
-Wire Wire Line
-	1550 2650 1250 2650
+	4100 4300 2500 4300
+Wire Wire Line
+	2600 4200 2600 2850
+Wire Wire Line
+	1250 2850 2600 2850
+Wire Wire Line
+	2500 4300 2500 2650
+Wire Wire Line
+	2500 2650 1250 2650
 $Comp
 L power:VDD #PWR04
@@
 	0    1    1    0
 $EndComp
-NoConn ~ 1700 2750
-Wire Wire Line
-	5700 3700 5700 2950
-Wire Wire Line
-	5700 2950 5100 2950
-Wire Wire Line
-	5750 3350 5750 3050
-Wire Wire Line
-	5750 3050 5100 3050
-Wire Wire Line
-	6250 3250 5100 3250
+Wire Wire Line
+	5900 3700 5900 2950
+Wire Wire Line
+	5800 3350 5800 3050
 Wire Wire Line
 	6250 2950 6250 3250
 Wire Wire Line
-	5100 3150 6150 3150
-Wire Wire Line
 	6150 3150 6150 2850
 Wire Wire Line
@@
 	5800 2550 5800 2650
 Wire Wire Line
-	5800 2650 5100 2650
-Wire Wire Line
-	5100 2750 6350 2750
-Wire Wire Line
 	5900 2650 5900 2850
 Wire Wire Line
-	5900 2850 5100 2850
-Wire Wire Line
-	1250 3850 1650 3850
-Wire Wire Line
-	1650 3850 1650 1600
-Wire Wire Line
-	1650 1600 5100 1600
-Wire Wire Line
-	5100 1600 5100 2550
-Wire Wire Line
-	1250 3350 1700 3350
-Wire Wire Line
-	1250 3450 1700 3450
-Wire Wire Line
-	1250 3750 1700 3750
-Wire Wire Line
-	1700 3750 1700 3650
-Wire Wire Line
-	5100 3350 5250 3350
-Wire Wire Line
-	5250 3350 5250 4400
-Wire Wire Line
-	5250 4400 1500 4400
-Wire Wire Line
-	1500 4400 1500 3650
-Wire Wire Line
-	1500 3650 1250 3650
-Wire Wire Line
-	1250 3550 1750 3550
-Wire Wire Line
-	1750 3550 1750 4450
-Wire Wire Line
-	1750 4450 5200 4450
-Wire Wire Line
-	5200 4450 5200 3450
-Wire Wire Line
-	5200 3450 5100 3450
+	1250 3850 2700 3850
+Wire Wire Line
+	2700 3850 2700 2300
+Wire Wire Line
+	2700 2300 3950 2300
+Wire Wire Line
+	3950 2300 3950 2550
+Wire Wire Line
+	1250 3750 2800 3750
+Wire Wire Line
+	2800 3750 2800 3650
+Wire Wire Line
+	4300 3350 4300 4500
+Wire Wire Line
+	4300 4500 2300 4500
+Wire Wire Line
+	2300 4500 2300 3650
+Wire Wire Line
+	2300 3650 1250 3650
+Wire Wire Line
+	1250 3550 2400 3550
+Wire Wire Line
+	2400 3550 2400 4400
+Wire Wire Line
+	2400 4400 4200 4400
+Wire Wire Line
+	4200 4400 4200 3450
+Wire Wire Line
+	3500 2050 3500 2350
+Wire Wire Line
+	3900 2650 5800 2650
+Wire Wire Line
+	3900 2750 6350 2750
+Wire Wire Line
+	3900 2850 5900 2850
+Wire Wire Line
+	3900 2950 5900 2950
+Wire Wire Line
+	3900 3250 6250 3250
+Wire Wire Line
+	3900 3350 4300 3350
+Wire Wire Line
+	3900 3450 4200 3450
+Wire Wire Line
+	4000 3650 3900 3650
+Wire Wire Line
+	3900 3150 6150 3150
+Wire Wire Line
+	3400 2050 3400 2350
+Wire Wire Line
+	3900 3550 4100 3550
+Wire Wire Line
+	3900 3050 5800 3050
+Wire Wire Line
+	3900 2550 3950 2550
+NoConn ~ 2900 2750
+Wire Wire Line
+	1250 2550 2900 2550
+Wire Wire Line
+	1250 3350 2900 3350
+Wire Wire Line
+	1250 3450 2900 3450
+Wire Wire Line
+	2800 3650 2900 3650
 $EndSCHEMATC

Commit message: Digit PCB is now 100% via-free!
Connections:
- wire segments 64 -> 72
Changed lines of the file:
@@
 	6150 2850 6350 2850
-Wire Wire Line
-	5800 2550 5800 2650
 Wire Wire Line
 	5900 2650 5900 2850
@@
 	3950 2300 3950 2550
 Wire Wire Line
-	1250 3750 2800 3750
-Wire Wire Line
-	2800 3750 2800 3650
-Wire Wire Line
 	4300 3350 4300 4500
-Wire Wire Line
-	4300 4500 2300 4500
-Wire Wire Line
-	2300 4500 2300 3650
-Wire Wire Line
-	2300 3650 1250 3650
-Wire Wire Line
-	1250 3550 2400 3550
-Wire Wire Line
-	2400 3550 2400 4400
-Wire Wire Line
-	2400 4400 4200 4400
 Wire Wire Line
 	4200 4400 4200 3450
 Wire Wire Line
 	3500 2050 3500 2350
-Wire Wire Line
-	3900 2650 5800 2650
 Wire Wire Line
 	3900 2750 6350 2750
@@
 	1250 2550 2900 2550
 Wire Wire Line
-	1250 3350 2900 3350
+	2900 3650 2800 3650
 Wire Wire Line
-	1250 3450 2900 3450
+	2800 3650 2800 2200
 Wire Wire Line
-	2800 3650 2900 3650
+	2800 2200 5800 2200
+Wire Wire Line
+	5800 2200 5800 2550
+Wire Wire Line
+	4400 4600 4400 2650
+Wire Wire Line
+	4400 2650 3900 2650
+Wire Wire Line
+	2300 3450 2300 3750
+Wire Wire Line
+	2300 3750 1250 3750
+Wire Wire Line
+	2300 3450 2900 3450
+Wire Wire Line
+	2200 3350 2200 3650
+Wire Wire Line
+	2200 3650 1250 3650
+Wire Wire Line
+	2200 3350 2900 3350
+Wire Wire Line
+	1900 4600 1900 3550
+Wire Wire Line
+	1900 3550 1250 3550
+Wire Wire Line
+	1900 4600 4400 4600
+Wire Wire Line
+	2000 4500 2000 3450
+Wire Wire Line
+	2000 3450 1250 3450
+Wire Wire Line
+	2000 4500 4300 4500
+Wire Wire Line
+	2100 4400 2100 3350
+Wire Wire Line
+	2100 3350 1250 3350
+Wire Wire Line
+	2100 4400 4200 4400
 $EndSCHEMATC

Commit message: Moved the pin headers closer to each other
Parts:
- J1: footprint Connector_PinHeader_2.54mm:PinHeader_1x09_P2.54mm_Horizontal -> Connector_PinHeader_2.54mm:PinHeader_1x09_P2.54mm_Vertical
- J2: footprint Connector_PinHeader_2.54mm:PinHeader_1x05_P2.54mm_Horizontal -> Connector_PinHeader_2.54mm:PinHeader_1x05_P2.54mm_Vertical
Changed lines of the file:
@@
 F 0 "J2" H 1006 3575 50  0000 C CNN
 F 1 "STM32_SWD" H 1006 3484 50  0000 C CNN
-F 2 "Connector_PinHeader_2.54mm:PinHeader_1x05_P2.54mm_Horizontal" H 1250 2950 50  0001 C CNN
+F 2 "Connector_PinHeader_2.54mm:PinHeader_1x05_P2.54mm_Vertical" H 1250 2950 50  0001 C CNN
 F 3 "" H 1250 2950 50  0001 C CNN
 	1    1250 2950
@@
 F 0 "J1" H 1156 4328 50  0000 C CNN
 F 1 "Conn_01x09_Male" H 1156 4237 50  0000 C CNN
-F 2 "Connector_PinHeader_2.54mm:PinHeader_1x09_P2.54mm_Horizontal" H 1050 3750 50  0001 C CNN
+F 2 "Connector_PinHeader_2.54mm:PinHeader_1x09_P2.54mm_Vertical" H 1050 3750 50  0001 C CNN
 F 3 "~" H 1050 3750 50  0001 C CNN
 	1    1050 3750
-	1    0    0    -1
+	1    0    0    1
 $EndComp
 Connection ~ 3400 2050

Commit message: Use a transistor array instead of two discrete transistors
Parts:
- Q1: value PZT2222A -> BC847BS; footprint Package_TO_SOT_SMD:SOT-223-3_TabPin2 -> Package_TO_SOT_SMD:SOT-363_SC-70-6; symbol Transistor_BJT:PZT2222A -> Transistor_BJT:BC847BS
- Q1: renamed from Q2; value PZT2222A -> BC847BS; footprint Package_TO_SOT_SMD:SOT-223-3_TabPin2 -> Package_TO_SOT_SMD:SOT-363_SC-70-6; symbol Transistor_BJT:PZT2222A -> Transistor_BJT:BC847BS
Connections:
- wire segments 72 -> 74
Changed lines of the file:
@@
 $EndComp
 $Comp
-L Transistor_BJT:PZT2222A Q1
+L Transistor_BJT:BC847BS Q1
 U 1 1 5AE75159
 P 7300 3350
 F 0 "Q1" H 7491 3396 50  0000 L CNN
-F 1 "PZT2222A" H 7491 3305 50  0000 L CNN
-F 2 "Package_TO_SOT_SMD:SOT-223-3_TabPin2" H 7500 3450 50  0001 C CNN
+F 1 "BC847BS" H 7491 3305 50  0000 L CNN
+F 2 "Package_TO_SOT_SMD:SOT-363_SC-70-6" H 7500 3450 50  0001 C CNN
 F 3 "" H 7300 3350 50  0001 C CNN
 	1    7300 3350
@@
 	7400 2750 7350 2750
 $Comp
-L Transistor_BJT:PZT2222A Q2
-U 1 1 5AE7533B
+L Transistor_BJT:BC847BS Q1
+U 2 1 5AE7533B
 P 7550 3700
-F 0 "Q2" H 7741 3746 50  0000 L CNN
-F 1 "PZT2222A" H 7741 3655 50  0000 L CNN
-F 2 "Package_TO_SOT_SMD:SOT-223-3_TabPin2" H 7750 3800 50  0001 C CNN
+F 0 "Q1" H 7741 3746 50  0000 L CNN
+F 1 "BC847BS" H 7741 3655 50  0000 L CNN
+F 2 "Package_TO_SOT_SMD:SOT-363_SC-70-6" H 7750 3800 50  0001 C CNN
 F 3 "" H 7550 3700 50  0001 C CNN
-	1    7550 3700
+	2    7550 3700
 	1    0    0    -1
 $EndComp
@@
 $EndComp
 Wire Wire Line
-	5900 3700 5900 2950
-Wire Wire Line
-	5800 3350 5800 3050
+	5900 3700 5900 3050
 Wire Wire Line
 	6250 2950 6250 3250
@@
 	6150 2850 6350 2850
 Wire Wire Line
-	5900 2650 5900 2850
-Wire Wire Line
 	1250 3850 2700 3850
 Wire Wire Line
@@
 	3500 2050 3500 2350
 Wire Wire Line
-	3900 2750 6350 2750
-Wire Wire Line
-	3900 2850 5900 2850
-Wire Wire Line
-	3900 2950 5900 2950
-Wire Wire Line
 	3900 3250 6250 3250
 Wire Wire Line
@@
 Wire Wire Line
 	3900 3550 4100 3550
-Wire Wire Line
-	3900 3050 5800 3050
 Wire Wire Line
 	3900 2550 3950 2550
@@
 Wire Wire Line
 	2100 4400 4200 4400
+Wire Wire Line
+	5900 2650 5900 2750
+Wire Wire Line
+	5900 2750 3900 2750
+Wire Wire Line
+	6350 2750 6000 2750
+Wire Wire Line
+	6000 2750 6000 2850
+Wire Wire Line
+	6000 2850 3900 2850
+Wire Wire Line
+	5800 2950 3900 2950
+Wire Wire Line
+	5800 2950 5800 3350
+Wire Wire Line
+	3900 3050 5900 3050
 $EndSCHEMATC
