File: pcb/button-node/button-node.kicad_pcb (KiCad board)
At the start: 2 copper layers, 30.5 x 27.9 mm, 10 parts, among them J1 STM32_SWD, J2 PicoTalk, SW1 Btn1, SW2 Btn2, SW3 Btn3, SW4 Btn4, U1 STM32F030F4Px

Commit message: Motherboard PCB
Routing:
- net GND: track 43.4 -> 30.2 mm
- net VDD: track 98.6 -> 103.2 mm
Other:
- outline, holes or cut-outs redrawn
- rule trace_min: 0.2 -> 0.4
- board text added: "PN Btn"
Changed lines of the file:
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@@
   (general
     (thickness 1.6)
-    (drawings 4)
-    (tracks 101)
+    (drawings 14)
+    (tracks 99)
     (zones 0)
     (modules 10)
@@
     (zone_clearance 0.508)
     (zone_45_only no)
-    (trace_min 0.2)
+    (trace_min 0.4)
     (segment_width 0.2)
     (edge_width 0.15)
@@
     )
   )
-  (gr_line (start 124.46 154.94) (end 124.46 127) (layer Edge.Cuts) (width 0.15))
-  (gr_line (start 154.94 154.94) (end 124.46 154.94) (layer Edge.Cuts) (width 0.15))
+  (gr_text "PN\nBtn" (at 127 140.97) (layer F.Cu)
+    (effects (font (size 1.5 1.5) (thickness 0.3)))
+  )
+  (gr_line (start 135.89 152.4) (end 143.51 152.4) (layer Edge.Cuts) (width 0.15))
+  (gr_line (start 133.35 154.94) (end 124.46 154.94) (layer Edge.Cuts) (width 0.15))
+  (gr_arc (start 143.51 154.94) (end 146.05 154.94) (angle -90) (layer Edge.Cuts) (width 0.15))
+  (gr_arc (start 135.89 154.94) (end 135.89 152.4) (angle -90) (layer Edge.Cuts) (width 0.15))
+  (gr_line (start 146.05 127) (end 154.94 127) (layer Edge.Cuts) (width 0.15))
+  (gr_line (start 137.16 130.81) (end 142.24 130.81) (layer Edge.Cuts) (width 0.15))
+  (gr_arc (start 142.24 127) (end 142.24 130.81) (angle -90) (layer Edge.Cuts) (width 0.15))
+  (gr_arc (start 137.16 127) (end 133.35 127) (angle -90) (layer Edge.Cuts) (width 0.15))
+  (gr_line (start 124.46 129.54) (end 127 127) (layer Edge.Cuts) (width 0.15))
+  (gr_line (start 124.46 154.94) (end 124.46 129.54) (layer Edge.Cuts) (width 0.15))
+  (gr_line (start 154.94 154.94) (end 146.05 154.94) (layer Edge.Cuts) (width 0.15))
   (gr_line (start 154.94 127) (end 154.94 154.94) (layer Edge.Cuts) (width 0.15))
-  (gr_line (start 124.46 127) (end 154.94 127) (layer Edge.Cuts) (width 0.15))
+  (gr_line (start 127 127) (end 133.35 127) (layer Edge.Cuts) (width 0.15))
   (segment (start 136.75 141.915) (end 142.65 141.915) (width 0.4) (layer F.Cu) (net 2))
   (segment (start 142.65 141.890001) (end 142.65 141.915) (width 0.4) (layer F.Cu) (net 2))
@@
   (segment (start 151.82 145.9) (end 151.82 147.314213) (width 0.4) (layer B.Cu) (net 2))
   (segment (start 127 136.04) (end 127 146.05) (width 0.4) (layer B.Cu) (net 2))
-  (segment (start 128.400001 128.139999) (end 127 129.54) (width 0.4) (layer B.Cu) (net 2))
-  (segment (start 147.32 129.54) (end 145.919999 128.139999) (width 0.4) (layer B.Cu) (net 2))
-  (segment (start 145.919999 128.139999) (end 128.400001 128.139999) (width 0.4) (layer B.Cu) (net 2))
   (segment (start 127 129.54) (end 127 136.04) (width 0.4) (layer B.Cu) (net 2))
   (segment (start 144.78 138.58) (end 147.32 136.04) (width 0.4) (layer F.Cu) (net 2))
@@
   (segment (start 134.62 139.7) (end 134.62 140.91) (width 0.4) (layer F.Cu) (net 2))
   (segment (start 134.62 139.7) (end 134.62 133.33) (width 0.4) (layer F.Cu) (net 2))
-  (segment (start 139.7 132.4625) (end 141.3525 130.81) (width 0.4) (layer F.Cu) (net 4))
+  (segment (start 150.820001 146.899999) (end 151.82 145.9) (width 0.4) (layer B.Cu) (net 2))
+  (segment (start 150.269999 147.450001) (end 150.820001 146.899999) (width 0.4) (layer B.Cu) (net 2))
+  (segment (start 128.400001 147.450001) (end 150.269999 147.450001) (width 0.4) (layer B.Cu) (net 2))
+  (segment (start 127 146.05) (end 128.400001 147.450001) (width 0.4) (layer B.Cu) (net 2))
   (segment (start 139.7 133.33) (end 139.7 132.4625) (width 0.4) (layer F.Cu) (net 4))
-  (segment (start 144.110002 130.81) (end 141.3525 130.81) (width 0.4) (layer F.Cu) (net 4))
-  (segment (start 149.86 136.559998) (end 144.110002 130.81) (width 0.4) (layer F.Cu) (net 4))
   (segment (start 149.86 138.8125) (end 149.86 136.559998) (width 0.4) (layer F.Cu) (net 4))
   (segment (start 149.600002 142.565) (end 143.775 142.565) (width 0.4) (layer F.Cu) (net 4))
@@
     (polygon
       (pts
-        (xy 124.46 127) (xy 154.94 127) (xy 154.94 154.94) (xy 124.46 154.94)
+        (xy 124.46 129.54) (xy 127 127) (xy 154.94 127) (xy 154.94 154.94) (xy 124.46 154.94)
       )
     )
@@
     (polygon
       (pts
-        (xy 124.46 127) (xy 154.94 127) (xy 154.94 154.94) (xy 124.46 154.94)
+        (xy 124.46 129.54) (xy 127 127) (xy 154.94 127) (xy 154.94 154.94) (xy 124.46 154.94)
       )
     )

Commit message: Pin orientation
Parts:
- J1, J2: moved to B.Cu
- turned J1 to 270 degrees
- turned J2 to 270 degrees
