File: pcb/motherboard/motherboard.kicad_pcb (KiCad board)
At the start: 2 copper layers, 160 x 96.5 mm, 40 parts, among them J1 UART, U1 Huzzah32, U2 LM317_3PinPackage

Commit message: Track cleanup
Routing:
- net GND: track 381.1 -> 344.3 mm
- added copper zone on F.Cu, net (none)
- removed copper zone on F.Cu, net GND
