File: pcb/motherboard/motherboard.kicad_pcb (KiCad board)
At the start: 2 copper layers, 160 x 96.5 mm, 40 parts, among them J1 UART, U1 Huzzah32, U2 LM317_3PinPackage

Commit message: Added status LEDs to motherboard
Parts:
- added D1: LED_Reset, LED_SMD:LED_0603_1608Metric_Pad0.82x1.00mm_HandSolder, F.Cu at (157.6, 49.5)
- added D2: LED_Vdd, LED_SMD:LED_0603_1608Metric_Pad0.82x1.00mm_HandSolder, F.Cu at (166.2, 49.5)
- added R1: 100, Resistor_SMD:R_0603_1608Metric_Pad0.99x1.00mm_HandSolder, F.Cu at (157.7, 53.3)
- added R12: 100, Resistor_SMD:R_0603_1608Metric_Pad0.99x1.00mm_HandSolder, F.Cu at (166.1, 53.3)
- renumbered R9 to R10, R10 to R11, R11 to R13, R12 to R14, R13 to R15, R14 to R16, R15 to R17, R16 to R18, R17 to R19, R1 to R2, R18 to R20, R19 to R21, R20 to R22, R21 to R23, R22 to R24, R23 to R25, R24 to R26, R25 to R27, R26 to R28, R2 to R3, R3 to R4, R4 to R5, R5 to R6, R6 to R7, R7 to R8, R8 to R9
Routing:
- net VDD: track 642.7 -> 659.1 mm, vias 3 -> 4
- net /nReset: track 319.2 -> 335.0 mm
- net GND: track 344.3 -> 350.9 mm, vias 0 -> 1
- net Net-(D1-Pad1): track 0.00 -> 4.47 mm
- net Net-(D2-Pad1): track 0.00 -> 3.81 mm
Other:
- board text added: "ON"
- board text added: "POWER"

Commit message: Make the DRC happy
Routing:
- net VDD: track 659.1 -> 659.9 mm
Changed lines of the file:
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@@
   (segment (start 185.42 52.45) (end 182.8825 49.9125) (width 0.4) (layer B.Cu) (net 2) (status 20))
   (segment (start 185.42 57.15) (end 185.42 52.45) (width 0.4) (layer B.Cu) (net 2) (status 10))
-  (segment (start 182.88 49.9125) (end 182.8775 49.9125) (width 0.4) (layer B.Cu) (net 2) (status 30))
   (segment (start 132.08 39.39) (end 132.08 40.64) (width 0.4) (layer B.Cu) (net 2) (status 20))
   (segment (start 134.64 36.83) (end 132.08 39.39) (width 0.4) (layer B.Cu) (net 2))
@@
   (segment (start 132.98 51.565) (end 104.14 51.565) (width 0.4) (layer B.Cu) (net 2))
   (segment (start 104.14 51.565) (end 100.349999 55.355001) (width 0.4) (layer B.Cu) (net 2))
-  (segment (start 182.8775 49.9125) (end 176.53 43.565) (width 0.4) (layer B.Cu) (net 2))
-  (segment (start 176.53 43.565) (end 169.795 36.83) (width 0.4) (layer B.Cu) (net 2))
-  (segment (start 165.1 36.83) (end 134.64 36.83) (width 0.4) (layer B.Cu) (net 2))
-  (segment (start 169.795 36.83) (end 165.1 36.83) (width 0.4) (layer B.Cu) (net 2))
-  (via (at 160.655 36.83) (size 1.8) (drill 0.55) (layers F.Cu B.Cu) (net 2))
-  (segment (start 160.655 47.708493) (end 160.655 36.83) (width 0.4) (layer F.Cu) (net 2))
   (segment (start 165.405 49.53) (end 162.476507 49.53) (width 0.4) (layer F.Cu) (net 2))
   (segment (start 162.476507 49.53) (end 160.655 47.708493) (width 0.4) (layer F.Cu) (net 2))
+  (segment (start 182.8775 49.9125) (end 182.88 49.9125) (width 0.4) (layer B.Cu) (net 2))
+  (segment (start 169.795 36.83) (end 182.8775 49.9125) (width 0.4) (layer B.Cu) (net 2))
+  (via (at 160.655 38.735) (size 1.8) (drill 0.55) (layers F.Cu B.Cu) (net 2))
+  (segment (start 160.655 47.708493) (end 160.655 38.735) (width 0.4) (layer F.Cu) (net 2))
+  (segment (start 160.655 38.735) (end 162.56 36.83) (width 0.4) (layer B.Cu) (net 2))
+  (segment (start 134.64 36.83) (end 162.56 36.83) (width 0.4) (layer B.Cu) (net 2))
+  (segment (start 162.56 36.83) (end 169.795 36.83) (width 0.4) (layer B.Cu) (net 2))
   (segment (start 67.31 74.93) (end 66.04 73.66) (width 0.4) (layer B.Cu) (net 3) (status 20))
   (segment (start 67.31 105.41) (end 67.31 74.93) (width 0.4) (layer B.Cu) (net 3))

Commit message: Various desperate troubleshooting
Parts:
- added R13: 820, Resistor_SMD:R_0603_1608Metric_Pad0.99x1.00mm_HandSolder, B.Cu at (169.3, 109.9)
- renumbered R13 to R14, R14 to R15, R15 to R16, R16 to R17, R17 to R18, R18 to R19, R19 to R20, R20 to R21, R21 to R22, R22 to R23, R23 to R24, R24 to R25, R25 to R26, R26 to R27, R27 to R28, R28 to R29
Routing:
- net GND: track 350.9 -> 356.9 mm
- net /nReset: track 335.0 -> 338.1 mm
