File: pcb/motherboard/motherboard.sch (KiCad schematic (older format))
At the start: 35 parts, among them J1 UART, U1 Huzzah32

Commit message: Bring our own voltage regulator instead of using the Huzzah32's built-in
Parts:
- added C1: 0.1µF, Capacitor_SMD:C_0603_1608Metric_Pad0.99x1.00mm_HandSolder, symbol device:C
- added C2: 1.0µF, Capacitor_SMD:C_0603_1608Metric_Pad0.99x1.00mm_HandSolder, symbol device:C
- added R15: 240, Resistor_SMD:R_0603_1608Metric_Pad0.99x1.00mm_HandSolder, symbol device:R
- added R16: 390, Resistor_SMD:R_0603_1608Metric_Pad0.99x1.00mm_HandSolder, symbol device:R
- added U2: LM317_3PinPackage, Package_TO_SOT_THT:TO-220-3_Vertical, symbol Regulator_Linear:LM317_3PinPackage
- renumbered R15 to R17, R16 to R18, R17 to R19, R18 to R20, R19 to R21, R20 to R22, R21 to R23, R22 to R24, R23 to R25, R24 to R26
Connections:
- net labels added: VBUS
- wire segments 121 -> 134
- no-connect marks 18 -> 19
Changed lines of the file:
@@
 $EndComp
 $Comp
-L power:VDD #PWR018
+L power:VDD #PWR021
 U 1 1 5AF195D5
 P 1400 4300
-F 0 "#PWR018" H 1400 4150 50  0001 C CNN
+F 0 "#PWR021" H 1400 4150 50  0001 C CNN
 F 1 "VDD" V 1418 4427 50  0000 L CNN
 F 2 "" H 1400 4300 50  0001 C CNN
@@
 $EndComp
 $Comp
-L power:VDD #PWR019
+L power:VDD #PWR022
 U 1 1 5AF197AB
 P 3350 4300
-F 0 "#PWR019" H 3350 4150 50  0001 C CNN
+F 0 "#PWR022" H 3350 4150 50  0001 C CNN
 F 1 "VDD" V 3368 4427 50  0000 L CNN
 F 2 "" H 3350 4300 50  0001 C CNN
@@
 $EndComp
 $Comp
-L power:VDD #PWR020
+L power:VDD #PWR023
 U 1 1 5AF19C08
 P 5200 4300
-F 0 "#PWR020" H 5200 4150 50  0001 C CNN
+F 0 "#PWR023" H 5200 4150 50  0001 C CNN
 F 1 "VDD" V 5218 4427 50  0000 L CNN
 F 2 "" H 5200 4300 50  0001 C CNN
@@
 $EndComp
 $Comp
-L power:GND #PWR021
+L power:GND #PWR024
 U 1 1 5AF1A2C4
 P 1400 4500
-F 0 "#PWR021" H 1400 4250 50  0001 C CNN
+F 0 "#PWR024" H 1400 4250 50  0001 C CNN
 F 1 "GND" V 1405 4372 50  0000 R CNN
 F 2 "" H 1400 4500 50  0001 C CNN
@@
 $EndComp
 $Comp
-L power:GND #PWR022
+L power:GND #PWR025
 U 1 1 5AF1A4E9
 P 3350 4500
-F 0 "#PWR022" H 3350 4250 50  0001 C CNN
+F 0 "#PWR025" H 3350 4250 50  0001 C CNN
 F 1 "GND" V 3355 4372 50  0000 R CNN
 F 2 "" H 3350 4500 50  0001 C CNN
@@
 $EndComp
 $Comp
-L power:GND #PWR023
+L power:GND #PWR026
 U 1 1 5AF1B6E8
 P 5200 4500
-F 0 "#PWR023" H 5200 4250 50  0001 C CNN
+F 0 "#PWR026" H 5200 4250 50  0001 C CNN
 F 1 "GND" V 5205 4372 50  0000 R CNN
 F 2 "" H 5200 4500 50  0001 C CNN
@@
 	5150 1400 6300 1400
 $Comp
-L device:R R15
+L device:R R17
 U 1 1 5AF30402
 P 2600 5200
-F 0 "R15" H 2670 5246 50  0000 L CNN
+F 0 "R17" H 2670 5246 50  0000 L CNN
 F 1 "4.7K" H 2670 5155 50  0000 L CNN
 F 2 "Resistor_SMD:R_0603_1608Metric_Pad0.99x1.00mm_HandSolder" V 2530 5200 50  0001 C CNN
@@
 	2600 4350 2600 5050
 $Comp
-L device:R R16
+L device:R R18
 U 1 1 5AF32114
 P 2900 5200
-F 0 "R16" H 2970 5246 50  0000 L CNN
+F 0 "R18" H 2970 5246 50  0000 L CNN
 F 1 "4.7K" H 2970 5155 50  0000 L CNN
 F 2 "Resistor_SMD:R_0603_1608Metric_Pad0.99x1.00mm_HandSolder" V 2830 5200 50  0001 C CNN
@@
 $EndComp
 $Comp
-L device:R R17
+L device:R R19
 U 1 1 5AF32150
 P 3200 5200
-F 0 "R17" H 3270 5246 50  0000 L CNN
+F 0 "R19" H 3270 5246 50  0000 L CNN
 F 1 "4.7K" H 3270 5155 50  0000 L CNN
 F 2 "Resistor_SMD:R_0603_1608Metric_Pad0.99x1.00mm_HandSolder" V 3130 5200 50  0001 C CNN
@@
 $EndComp
 $Comp
-L device:R R18
+L device:R R20
 U 1 1 5AF321F4
 P 3500 5200
-F 0 "R18" H 3570 5246 50  0000 L CNN
+F 0 "R20" H 3570 5246 50  0000 L CNN
 F 1 "4.7K" H 3570 5155 50  0000 L CNN
 F 2 "Resistor_SMD:R_0603_1608Metric_Pad0.99x1.00mm_HandSolder" V 3430 5200 50  0001 C CNN
@@
 Connection ~ 3000 4650
 $Comp
-L device:R R19
+L device:R R21
 U 1 1 5AF3B1F0
 P 4350 5200
-F 0 "R19" H 4420 5246 50  0000 L CNN
+F 0 "R21" H 4420 5246 50  0000 L CNN
 F 1 "4.7K" H 4420 5155 50  0000 L CNN
 F 2 "Resistor_SMD:R_0603_1608Metric_Pad0.99x1.00mm_HandSolder" V 4280 5200 50  0001 C CNN
@@
 $EndComp
 $Comp
-L device:R R20
+L device:R R22
 U 1 1 5AF3D1B1
 P 4650 5200
-F 0 "R20" H 4720 5246 50  0000 L CNN
+F 0 "R22" H 4720 5246 50  0000 L CNN
 F 1 "4.7K" H 4720 5155 50  0000 L CNN
 F 2 "Resistor_SMD:R_0603_1608Metric_Pad0.99x1.00mm_HandSolder" V 4580 5200 50  0001 C CNN
@@
 $EndComp
 $Comp
-L device:R R21
+L device:R R23
 U 1 1 5AF3D263
 P 4950 5200
-F 0 "R21" H 5020 5246 50  0000 L CNN
+F 0 "R23" H 5020 5246 50  0000 L CNN
 F 1 "4.7K" H 5020 5155 50  0000 L CNN
 F 2 "Resistor_SMD:R_0603_1608Metric_Pad0.99x1.00mm_HandSolder" V 4880 5200 50  0001 C CNN
@@
 	4650 5350 4950 5350
 $Comp
-L power:VDD #PWR024
+L power:VDD #PWR027
 U 1 1 5AF43D0B
 P 2900 5350
-F 0 "#PWR024" H 2900 5200 50  0001 C CNN
+F 0 "#PWR027" H 2900 5200 50  0001 C CNN
 F 1 "VDD" H 2918 5523 50  0000 C CNN
 F 2 "" H 2900 5350 50  0001 C CNN
@@
 Connection ~ 5150 800
 $Comp
-L device:R R22
+L device:R R24
 U 1 1 5AF53FDF
 P 6550 5200
-F 0 "R22" H 6620 5246 50  0000 L CNN
+F 0 "R24" H 6620 5246 50  0000 L CNN
 F 1 "4.7K" H 6620 5155 50  0000 L CNN
 F 2 "Resistor_SMD:R_0603_1608Metric_Pad0.99x1.00mm_HandSolder" V 6480 5200 50  0001 C CNN
@@
 $EndComp
 $Comp
-L device:R R24
+L device:R R26
 U 1 1 5AF54079
 P 7150 5200
-F 0 "R24" H 7220 5246 50  0000 L CNN
+F 0 "R26" H 7220 5246 50  0000 L CNN
 F 1 "4.7K" H 7220 5155 50  0000 L CNN
 F 2 "Resistor_SMD:R_0603_1608Metric_Pad0.99x1.00mm_HandSolder" V 7080 5200 50  0001 C CNN
@@
 	4350 4350 4350 5050
 $Comp
-L device:R R23
+L device:R R25
 U 1 1 5AF85C2C
 P 6850 5200
-F 0 "R23" H 6920 5246 50  0000 L CNN
+F 0 "R25" H 6920 5246 50  0000 L CNN
 F 1 "4.7K" H 6920 5155 50  0000 L CNN
 F 2 "Resistor_SMD:R_0603_1608Metric_Pad0.99x1.00mm_HandSolder" V 6780 5200 50  0001 C CNN
@@
 	6850 5350 7150 5350
 Connection ~ 6850 5350
-$Comp
-L power:VDD #PWR08
-U 1 1 5AF26C1B
-P 8400 1900
-F 0 "#PWR08" H 8400 1750 50  0001 C CNN
-F 1 "VDD" H 8417 2073 50  0000 C CNN
-F 2 "" H 8400 1900 50  0001 C CNN
-F 3 "" H 8400 1900 50  0001 C CNN
-	1    8400 1900
-	1    0    0    -1
-$EndComp
 $Comp
 L power:GND #PWR011
@@
 Text Label 9000 2100 0    50   ~ 0
 TX
+$Comp
+L power:VBUS #PWR08
+U 1 1 5AFE8DC5
+P 8300 1900
+F 0 "#PWR08" H 8300 1750 50  0001 C CNN
+F 1 "VBUS" H 8315 2073 50  0000 C CNN
+F 2 "" H 8300 1900 50  0001 C CNN
+F 3 "" H 8300 1900 50  0001 C CNN
+	1    8300 1900
+	1    0    0    -1
+$EndComp
+NoConn ~ 8400 1900
+$Comp
+L Regulator_Linear:LM317_3PinPackage U2
+U 1 1 5AFF1E1E
+P 8400 3650
+F 0 "U2" H 8400 3892 50  0000 C CNN
+F 1 "LM317_3PinPackage" H 8400 3801 50  0000 C CNN
+F 2 "Package_TO_SOT_THT:TO-220-3_Vertical" H 8400 3900 50  0001 C CIN
+F 3 "http://www.ti.com/lit/ds/symlink/lm317.pdf" H 8400 3650 50  0001 C CNN
+	1    8400 3650
+	1    0    0    -1
+$EndComp
+$Comp
+L power:VBUS #PWR018
+U 1 1 5AFF2111
+P 7900 3650
+F 0 "#PWR018" H 7900 3500 50  0001 C CNN
+F 1 "VBUS" V 7915 3777 50  0000 L CNN
+F 2 "" H 7900 3650 50  0001 C CNN
+F 3 "" H 7900 3650 50  0001 C CNN
+	1    7900 3650
+	0    -1   -1   0
+$EndComp
+$Comp
+L power:VDD #PWR019
+U 1 1 5AFF2258
+P 9300 3650
+F 0 "#PWR019" H 9300 3500 50  0001 C CNN
+F 1 "VDD" V 9317 3778 50  0000 L CNN
+F 2 "" H 9300 3650 50  0001 C CNN
+F 3 "" H 9300 3650 50  0001 C CNN
+	1    9300 3650
+	0    1    1    0
+$EndComp
+$Comp
+L device:C C1
+U 1 1 5AFF257B
+P 8000 4000
+F 0 "C1" H 8115 4046 50  0000 L CNN
+F 1 "0.1µF" H 8115 3955 50  0000 L CNN
+F 2 "Capacitor_SMD:C_0603_1608Metric_Pad0.99x1.00mm_HandSolder" H 8038 3850 50  0001 C CNN
+F 3 "" H 8000 4000 50  0001 C CNN
+	1    8000 4000
+	1    0    0    -1
+$EndComp
+Wire Wire Line
+	8000 3650 8100 3650
+Wire Wire Line
+	7900 3650 8000 3650
+Connection ~ 8000 3650
+Wire Wire Line
+	8000 3850 8000 3650
+$Comp
+L device:R R15
+U 1 1 5B007F1E
+P 8850 3800
+F 0 "R15" H 8920 3846 50  0000 L CNN
+F 1 "240" H 8920 3755 50  0000 L CNN
+F 2 "Resistor_SMD:R_0603_1608Metric_Pad0.99x1.00mm_HandSolder" V 8780 3800 50  0001 C CNN
+F 3 "" H 8850 3800 50  0001 C CNN
+	1    8850 3800
+	1    0    0    -1
+$EndComp
+Wire Wire Line
+	8700 3650 8850 3650
+$Comp
+L device:C C2
+U 1 1 5B00C5A8
+P 9150 4000
+F 0 "C2" H 9265 4046 50  0000 L CNN
+F 1 "1.0µF" H 9265 3955 50  0000 L CNN
+F 2 "Capacitor_SMD:C_0603_1608Metric_Pad0.99x1.00mm_HandSolder" H 9188 3850 50  0001 C CNN
+F 3 "" H 9150 4000 50  0001 C CNN
+	1    9150 4000
+	1    0    0    -1
+$EndComp
+Wire Wire Line
+	8850 3650 9150 3650
+Connection ~ 8850 3650
+Connection ~ 9150 3650
+Wire Wire Line
+	9150 3650 9300 3650
+Wire Wire Line
+	9150 3850 9150 3650
+$Comp
+L device:R R16
+U 1 1 5B01EA63
+P 8600 4100
+F 0 "R16" H 8670 4146 50  0000 L CNN
+F 1 "390" H 8670 4055 50  0000 L CNN
+F 2 "Resistor_SMD:R_0603_1608Metric_Pad0.99x1.00mm_HandSolder" V 8530 4100 50  0001 C CNN
+F 3 "" H 8600 4100 50  0001 C CNN
+	1    8600 4100
+	1    0    0    -1
+$EndComp
+Wire Wire Line
+	8000 4150 8000 4250
+Wire Wire Line
+	9150 4250 9150 4150
+$Comp
+L power:GND #PWR020
+U 1 1 5B0284A8
+P 8600 4250
+F 0 "#PWR020" H 8600 4000 50  0001 C CNN
+F 1 "GND" H 8605 4077 50  0000 C CNN
+F 2 "" H 8600 4250 50  0001 C CNN
+F 3 "" H 8600 4250 50  0001 C CNN
+	1    8600 4250
+	1    0    0    -1
+$EndComp
+Wire Wire Line
+	8400 3950 8600 3950
+Wire Wire Line
+	8000 4250 8600 4250
+Connection ~ 8600 4250
+Connection ~ 8600 3950
+Wire Wire Line
+	8600 3950 8850 3950
+Wire Wire Line
+	8600 4250 9150 4250
 $EndSCHEMATC

Commit message: Added status LEDs to motherboard
Parts:
- added D1: LED_Reset, LED_SMD:LED_0603_1608Metric_Pad0.82x1.00mm_HandSolder, symbol device:LED
- added D2: LED_Vdd, LED_SMD:LED_0603_1608Metric_Pad0.82x1.00mm_HandSolder, symbol device:LED
- added R1, R12: 100, Resistor_SMD:R_0603_1608Metric_Pad0.99x1.00mm_HandSolder, symbol device:R
- renumbered R9 to R10, R10 to R11, R11 to R13, R12 to R14, R13 to R15, R14 to R16, R15 to R17, R16 to R18, R17 to R19, R1 to R2, R18 to R20, R19 to R21, R20 to R22, R21 to R23, R22 to R24, R23 to R25, R24 to R26, R25 to R27, R26 to R28, R2 to R3, R3 to R4, R4 to R5, R5 to R6, R6 to R7, R7 to R8, R8 to R9
Connections:
- wire segments 134 -> 137

Commit message: Various desperate troubleshooting
Parts:
- added R13: 820, Resistor_SMD:R_0603_1608Metric_Pad0.99x1.00mm_HandSolder, symbol device:R
- renumbered R13 to R14, R14 to R15, R15 to R16, R16 to R17, R17 to R18, R18 to R19, R19 to R20, R20 to R21, R21 to R22, R22 to R23, R23 to R24, R24 to R25, R25 to R26, R26 to R27, R27 to R28, R28 to R29
Changed lines of the file:
@@
 $EndComp
 $Comp
-L power:VDD #PWR014
+L power:VDD #PWR015
 U 1 1 5AF19462
 P 1400 3000
-F 0 "#PWR014" H 1400 2850 50  0001 C CNN
+F 0 "#PWR015" H 1400 2850 50  0001 C CNN
 F 1 "VDD" V 1418 3127 50  0000 L CNN
 F 2 "" H 1400 3000 50  0001 C CNN
@@
 $EndComp
 $Comp
-L power:VDD #PWR023
+L power:VDD #PWR024
 U 1 1 5AF195D5
 P 1400 4300
-F 0 "#PWR023" H 1400 4150 50  0001 C CNN
+F 0 "#PWR024" H 1400 4150 50  0001 C CNN
 F 1 "VDD" V 1418 4427 50  0000 L CNN
 F 2 "" H 1400 4300 50  0001 C CNN
@@
 $EndComp
 $Comp
-L power:VDD #PWR024
+L power:VDD #PWR025
 U 1 1 5AF197AB
 P 3350 4300
-F 0 "#PWR024" H 3350 4150 50  0001 C CNN
+F 0 "#PWR025" H 3350 4150 50  0001 C CNN
 F 1 "VDD" V 3368 4427 50  0000 L CNN
 F 2 "" H 3350 4300 50  0001 C CNN
@@
 $EndComp
 $Comp
-L power:VDD #PWR015
+L power:VDD #PWR016
 U 1 1 5AF197C8
 P 3350 3000
-F 0 "#PWR015" H 3350 2850 50  0001 C CNN
+F 0 "#PWR016" H 3350 2850 50  0001 C CNN
 F 1 "VDD" V 3368 3127 50  0000 L CNN
 F 2 "" H 3350 3000 50  0001 C CNN
@@
 $EndComp
 $Comp
-L power:VDD #PWR016
+L power:VDD #PWR017
 U 1 1 5AF19B0A
 P 5200 3000
-F 0 "#PWR016" H 5200 2850 50  0001 C CNN
+F 0 "#PWR017" H 5200 2850 50  0001 C CNN
 F 1 "VDD" V 5218 3127 50  0000 L CNN
 F 2 "" H 5200 3000 50  0001 C CNN
@@
 $EndComp
 $Comp
-L power:VDD #PWR025
+L power:VDD #PWR026
 U 1 1 5AF19C08
 P 5200 4300
-F 0 "#PWR025" H 5200 4150 50  0001 C CNN
+F 0 "#PWR026" H 5200 4150 50  0001 C CNN
 F 1 "VDD" V 5218 4427 50  0000 L CNN
 F 2 "" H 5200 4300 50  0001 C CNN
@@
 $EndComp
 $Comp
-L power:GND #PWR026
+L power:GND #PWR027
 U 1 1 5AF1A2C4
 P 1400 4500
-F 0 "#PWR026" H 1400 4250 50  0001 C CNN
+F 0 "#PWR027" H 1400 4250 50  0001 C CNN
 F 1 "GND" V 1405 4372 50  0000 R CNN
 F 2 "" H 1400 4500 50  0001 C CNN
@@
 $EndComp
 $Comp
-L power:GND #PWR017
+L power:GND #PWR018
 U 1 1 5AF1A2F1
 P 1400 3200
-F 0 "#PWR017" H 1400 2950 50  0001 C CNN
+F 0 "#PWR018" H 1400 2950 50  0001 C CNN
 F 1 "GND" V 1405 3072 50  0000 R CNN
 F 2 "" H 1400 3200 50  0001 C CNN
@@
 $EndComp
 $Comp
-L power:GND #PWR018
+L power:GND #PWR019
 U 1 1 5AF1A4CC
 P 3350 3200
-F 0 "#PWR018" H 3350 2950 50  0001 C CNN
+F 0 "#PWR019" H 3350 2950 50  0001 C CNN
 F 1 "GND" V 3355 3072 50  0000 R CNN
 F 2 "" H 3350 3200 50  0001 C CNN
@@
 $EndComp
 $Comp
-L power:GND #PWR027
+L power:GND #PWR028
 U 1 1 5AF1A4E9
 P 3350 4500
-F 0 "#PWR027" H 3350 4250 50  0001 C CNN
+F 0 "#PWR028" H 3350 4250 50  0001 C CNN
 F 1 "GND" V 3355 4372 50  0000 R CNN
 F 2 "" H 3350 4500 50  0001 C CNN
@@
 $EndComp
 $Comp
-L power:GND #PWR019
+L power:GND #PWR020
 U 1 1 5AF1B509
 P 5200 3200
-F 0 "#PWR019" H 5200 2950 50  0001 C CNN
+F 0 "#PWR020" H 5200 2950 50  0001 C CNN
 F 1 "GND" V 5205 3072 50  0000 R CNN
 F 2 "" H 5200 3200 50  0001 C CNN
@@
 $EndComp
 $Comp
-L power:GND #PWR028
+L power:GND #PWR029
 U 1 1 5AF1B6E8
 P 5200 4500
-F 0 "#PWR028" H 5200 4250 50  0001 C CNN
+F 0 "#PWR029" H 5200 4250 50  0001 C CNN
 F 1 "GND" V 5205 4372 50  0000 R CNN
 F 2 "" H 5200 4500 50  0001 C CNN
@@
 	5150 1400 6300 1400
 $Comp
-L device:R R19
+L device:R R20
 U 1 1 5AF30402
 P 2600 5200
-F 0 "R19" H 2670 5246 50  0000 L CNN
+F 0 "R20" H 2670 5246 50  0000 L CNN
 F 1 "4.7K" H 2670 5155 50  0000 L CNN
 F 2 "Resistor_SMD:R_0603_1608Metric_Pad0.99x1.00mm_HandSolder" V 2530 5200 50  0001 C CNN
@@
 	2600 4350 2600 5050
 $Comp
-L device:R R20
+L device:R R21
 U 1 1 5AF32114
 P 2900 5200
-F 0 "R20" H 2970 5246 50  0000 L CNN
+F 0 "R21" H 2970 5246 50  0000 L CNN
 F 1 "4.7K" H 2970 5155 50  0000 L CNN
 F 2 "Resistor_SMD:R_0603_1608Metric_Pad0.99x1.00mm_HandSolder" V 2830 5200 50  0001 C CNN
@@
 $EndComp
 $Comp
-L device:R R21
+L device:R R22
 U 1 1 5AF32150
 P 3200 5200
-F 0 "R21" H 3270 5246 50  0000 L CNN
+F 0 "R22" H 3270 5246 50  0000 L CNN
 F 1 "4.7K" H 3270 5155 50  0000 L CNN
 F 2 "Resistor_SMD:R_0603_1608Metric_Pad0.99x1.00mm_HandSolder" V 3130 5200 50  0001 C CNN
@@
 $EndComp
 $Comp
-L device:R R22
+L device:R R23
 U 1 1 5AF321F4
 P 3500 5200
-F 0 "R22" H 3570 5246 50  0000 L CNN
+F 0 "R23" H 3570 5246 50  0000 L CNN
 F 1 "4.7K" H 3570 5155 50  0000 L CNN
 F 2 "Resistor_SMD:R_0603_1608Metric_Pad0.99x1.00mm_HandSolder" V 3430 5200 50  0001 C CNN
@@
 Connection ~ 3000 4650
 $Comp
-L device:R R23
+L device:R R24
 U 1 1 5AF3B1F0
 P 4350 5200
-F 0 "R23" H 4420 5246 50  0000 L CNN
+F 0 "R24" H 4420 5246 50  0000 L CNN
 F 1 "4.7K" H 4420 5155 50  0000 L CNN
 F 2 "Resistor_SMD:R_0603_1608Metric_Pad0.99x1.00mm_HandSolder" V 4280 5200 50  0001 C CNN
@@
 $EndComp
 $Comp
-L device:R R24
+L device:R R25
 U 1 1 5AF3D1B1
 P 4650 5200
-F 0 "R24" H 4720 5246 50  0000 L CNN
+F 0 "R25" H 4720 5246 50  0000 L CNN
 F 1 "4.7K" H 4720 5155 50  0000 L CNN
 F 2 "Resistor_SMD:R_0603_1608Metric_Pad0.99x1.00mm_HandSolder" V 4580 5200 50  0001 C CNN
@@
 $EndComp
 $Comp
-L device:R R25
+L device:R R26
 U 1 1 5AF3D263
 P 4950 5200
-F 0 "R25" H 5020 5246 50  0000 L CNN
+F 0 "R26" H 5020 5246 50  0000 L CNN
 F 1 "4.7K" H 5020 5155 50  0000 L CNN
 F 2 "Resistor_SMD:R_0603_1608Metric_Pad0.99x1.00mm_HandSolder" V 4880 5200 50  0001 C CNN
@@
 	4650 5350 4950 5350
 $Comp
-L power:VDD #PWR029
+L power:VDD #PWR030
 U 1 1 5AF43D0B
 P 2900 5350
-F 0 "#PWR029" H 2900 5200 50  0001 C CNN
+F 0 "#PWR030" H 2900 5200 50  0001 C CNN
 F 1 "VDD" H 2918 5523 50  0000 C CNN
 F 2 "" H 2900 5350 50  0001 C CNN
@@
 $EndComp
 $Comp
-L device:R R14
+L device:R R15
 U 1 1 5AF441A3
 P 3100 2550
-F 0 "R14" H 3170 2596 50  0000 L CNN
+F 0 "R15" H 3170 2596 50  0000 L CNN
 F 1 "4.7K" H 3170 2505 50  0000 L CNN
 F 2 "Resistor_SMD:R_0603_1608Metric_Pad0.99x1.00mm_HandSolder" V 3030 2550 50  0001 C CNN
@@
 	3100 2700 4700 2700
 $Comp
-L device:R R13
+L device:R R14
 U 1 1 5AF4424F
 P 2800 2550
-F 0 "R13" H 2870 2596 50  0000 L CNN
+F 0 "R14" H 2870 2596 50  0000 L CNN
 F 1 "4.7K" H 2870 2505 50  0000 L CNN
 F 2 "Resistor_SMD:R_0603_1608Metric_Pad0.99x1.00mm_HandSolder" V 2730 2550 50  0001 C CNN
@@
 Connection ~ 5150 800
 $Comp
-L device:R R26
+L device:R R27
 U 1 1 5AF53FDF
 P 6550 5200
-F 0 "R26" H 6620 5246 50  0000 L CNN
+F 0 "R27" H 6620 5246 50  0000 L CNN
 F 1 "4.7K" H 6620 5155 50  0000 L CNN
 F 2 "Resistor_SMD:R_0603_1608Metric_Pad0.99x1.00mm_HandSolder" V 6480 5200 50  0001 C CNN
@@
 $EndComp
 $Comp
-L device:R R28
+L device:R R29
 U 1 1 5AF54079
 P 7150 5200
-F 0 "R28" H 7220 5246 50  0000 L CNN
+F 0 "R29" H 7220 5246 50  0000 L CNN
 F 1 "4.7K" H 7220 5155 50  0000 L CNN
 F 2 "Resistor_SMD:R_0603_1608Metric_Pad0.99x1.00mm_HandSolder" V 7080 5200 50  0001 C CNN
@@
 	6550 5350 4950 5350
 $Comp
-L device:R R15
+L device:R R16
 U 1 1 5AF620FE
 P 6250 2550
-F 0 "R15" H 6320 2596 50  0000 L CNN
+F 0 "R16" H 6320 2596 50  0000 L CNN
 F 1 "4.7K" H 6320 2505 50  0000 L CNN
 F 2 "Resistor_SMD:R_0603_1608Metric_Pad0.99x1.00mm_HandSolder" V 6180 2550 50  0001 C CNN
@@
 	6250 2700 6400 2700
 $Comp
-L device:R R16
+L device:R R17
 U 1 1 5AF6220C
 P 6600 2550
-F 0 "R16" H 6670 2596 50  0000 L CNN
+F 0 "R17" H 6670 2596 50  0000 L CNN
 F 1 "4.7K" H 6670 2505 50  0000 L CNN
 F 2 "Resistor_SMD:R_0603_1608Metric_Pad0.99x1.00mm_HandSolder" V 6530 2550 50  0001 C CNN
@@
 	4350 4350 4350 5050
 $Comp
-L device:R R27
+L device:R R28
 U 1 1 5AF85C2C
 P 6850 5200
-F 0 "R27" H 6920 5246 50  0000 L CNN
+F 0 "R28" H 6920 5246 50  0000 L CNN
 F 1 "4.7K" H 6920 5155 50  0000 L CNN
 F 2 "Resistor_SMD:R_0603_1608Metric_Pad0.99x1.00mm_HandSolder" V 6780 5200 50  0001 C CNN
@@
 $EndComp
 $Comp
-L power:VBUS #PWR020
+L power:VBUS #PWR021
 U 1 1 5AFF2111
 P 7900 3650
-F 0 "#PWR020" H 7900 3500 50  0001 C CNN
+F 0 "#PWR021" H 7900 3500 50  0001 C CNN
 F 1 "VBUS" V 7915 3777 50  0000 L CNN
 F 2 "" H 7900 3650 50  0001 C CNN
@@
 $EndComp
 $Comp
-L power:VDD #PWR021
+L power:VDD #PWR022
 U 1 1 5AFF2258
 P 9300 3650
-F 0 "#PWR021" H 9300 3500 50  0001 C CNN
+F 0 "#PWR022" H 9300 3500 50  0001 C CNN
 F 1 "VDD" V 9317 3778 50  0000 L CNN
 F 2 "" H 9300 3650 50  0001 C CNN
@@
 	8000 3850 8000 3650
 $Comp
-L device:R R17
+L device:R R18
 U 1 1 5B007F1E
 P 8850 3800
-F 0 "R17" H 8920 3846 50  0000 L CNN
+F 0 "R18" H 8920 3846 50  0000 L CNN
 F 1 "240" H 8920 3755 50  0000 L CNN
 F 2 "Resistor_SMD:R_0603_1608Metric_Pad0.99x1.00mm_HandSolder" V 8780 3800 50  0001 C CNN
@@
 	9150 3850 9150 3650
 $Comp
-L device:R R18
+L device:R R19
 U 1 1 5B01EA63
 P 8600 4100
-F 0 "R18" H 8670 4146 50  0000 L CNN
+F 0 "R19" H 8670 4146 50  0000 L CNN
 F 1 "390" H 8670 4055 50  0000 L CNN
 F 2 "Resistor_SMD:R_0603_1608Metric_Pad0.99x1.00mm_HandSolder" V 8530 4100 50  0001 C CNN
@@
 	9150 4250 9150 4150
 $Comp
-L power:GND #PWR022
+L power:GND #PWR023
 U 1 1 5B0284A8
 P 8600 4250
-F 0 "#PWR022" H 8600 4000 50  0001 C CNN
+F 0 "#PWR023" H 8600 4000 50  0001 C CNN
 F 1 "GND" H 8605 4077 50  0000 C CNN
 F 2 "" H 8600 4250 50  0001 C CNN
@@
 Wire Wire Line
 	8800 1100 8800 900
+$Comp
+L device:R R13
+U 1 1 5B03393C
+P 8700 2500
+F 0 "R13" H 8770 2546 50  0000 L CNN
+F 1 "820" H 8770 2455 50  0000 L CNN
+F 2 "Resistor_SMD:R_0603_1608Metric_Pad0.99x1.00mm_HandSolder" V 8630 2500 50  0001 C CNN
+F 3 "" H 8700 2500 50  0001 C CNN
+F 4 "ESP32 also uses this pin for voltage detection" H 8700 2500 50  0001 C CNN "Rationale"
+	1    8700 2500
+	1    0    0    -1
+$EndComp
+Connection ~ 8700 2350
+$Comp
+L power:GND #PWR014
+U 1 1 5B033A3A
+P 8700 2650
+F 0 "#PWR014" H 8700 2400 50  0001 C CNN
+F 1 "GND" H 8705 2477 50  0000 C CNN
+F 2 "" H 8700 2650 50  0001 C CNN
+F 3 "" H 8700 2650 50  0001 C CNN
+	1    8700 2650
+	1    0    0    -1
+$EndComp
 $EndSCHEMATC
