File: pcb/led-node/led-node.kicad_pcb (KiCad board)
At the start: 2 copper layers, 30.5 x 27.9 mm, 12 parts, among them J1 STM32_SWD, J2 PicoTalk, U1 STM32F030F4Px

Commit message: Motherboard PCB
Parts:
- moved D2 3.89 mm to (131.3, 149.9)
- moved D4 3.81 mm to (147.3, 149.9)
- moved D1 0.80 mm to (131.3, 143.5)
- moved R1 0.80 mm to (127.5, 143.5)
Routing:
- net GND: track 63.4 -> 1.81 mm
- net Net-(D4-Pad2): track 4.56 -> 8.46 mm
- net Net-(D3-Pad1): track 4.75 -> 8.56 mm
- net Net-(D1-Pad1): track 4.75 -> 8.56 mm
- net Net-(D2-Pad2): track 5.03 -> 7.94 mm
- net Net-(D1-Pad2): track 4.02 -> 4.82 mm
Other:
- outline, holes or cut-outs redrawn
- board text added: "Pico Node LED"
Changed lines of the file:
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@@
   (general
     (thickness 1.6)
-    (drawings 4)
-    (tracks 85)
+    (drawings 14)
+    (tracks 67)
     (zones 0)
     (modules 12)
@@
   )
   (module LED_SMD:LED_0603_1608Metric (layer F.Cu)
-    (at 147.32 146.05 180)
+    (at 147.32 149.86 180)
     (descr "LED SMD 0603 (1608 Metric), square (rectangular) end terminal, IPC_7351 nominal, (Body size source: http://www.tortai-tech.com/upload/download/2011102023233369053.pdf), generated with kicad-footprint-generator")
     (tags diode)
@@
   )
   (module LED_SMD:LED_0603_1608Metric (layer F.Cu)
-    (at 132.08 146.05)
+    (at 131.28 149.86)
     (descr "LED SMD 0603 (1608 Metric), square (rectangular) end terminal, IPC_7351 nominal, (Body size source: http://www.tortai-tech.com/upload/download/2011102023233369053.pdf), generated with kicad-footprint-generator")
     (tags diode)
@@
   )
   (module LED_SMD:LED_0603_1608Metric (layer F.Cu)
-    (at 132.08 143.51)
+    (at 131.28 143.51)
     (descr "LED SMD 0603 (1608 Metric), square (rectangular) end terminal, IPC_7351 nominal, (Body size source: http://www.tortai-tech.com/upload/download/2011102023233369053.pdf), generated with kicad-footprint-generator")
     (tags diode)
@@
   )
   (module Resistor_SMD:R_0603_1608Metric (layer F.Cu)
-    (at 128.27 143.51 180)
+    (at 127.47 143.51 180)
     (descr "Resistor SMD 0603 (1608 Metric), square (rectangular) end terminal, IPC_7351 nominal, (Body size source: http://www.tortai-tech.com/upload/download/2011102023233369053.pdf), generated with kicad-footprint-generator")
     (tags resistor)
@@
     )
   )
-  (gr_line (start 124.46 154.94) (end 124.46 127) (layer Edge.Cuts) (width 0.15))
-  (gr_line (start 154.94 154.94) (end 124.46 154.94) (layer Edge.Cuts) (width 0.15))
+  (gr_text "Pico\nNode\nLED" (at 125.73 133.35) (layer F.Cu)
+    (effects (font (size 1.5 1.5) (thickness 0.3)) (justify left))
+  )
+  (gr_line (start 133.35 154.94) (end 124.46 154.94) (layer Edge.Cuts) (width 0.15))
+  (gr_line (start 135.89 152.4) (end 144.78 152.4) (layer Edge.Cuts) (width 0.15))
+  (gr_arc (start 144.78 154.94) (end 147.32 154.94) (angle -90) (layer Edge.Cuts) (width 0.15))
+  (gr_arc (start 135.89 154.94) (end 135.89 152.4) (angle -90) (layer Edge.Cuts) (width 0.15))
+  (gr_line (start 147.32 127) (end 154.94 127) (layer Edge.Cuts) (width 0.15))
+  (gr_line (start 137.16 130.81) (end 143.51 130.81) (layer Edge.Cuts) (width 0.15))
+  (gr_arc (start 143.51 127) (end 143.51 130.81) (angle -90) (layer Edge.Cuts) (width 0.2))
+  (gr_arc (start 137.16 127) (end 133.35 127) (angle -90) (layer Edge.Cuts) (width 0.2))
+  (gr_line (start 124.46 129.54) (end 127 127) (layer Edge.Cuts) (width 0.15))
+  (gr_line (start 124.46 154.94) (end 124.46 129.54) (layer Edge.Cuts) (width 0.15))
+  (gr_line (start 154.94 154.94) (end 147.32 154.94) (layer Edge.Cuts) (width 0.15))
   (gr_line (start 154.94 127) (end 154.94 154.94) (layer Edge.Cuts) (width 0.15))
-  (gr_line (start 124.46 127) (end 154.94 127) (layer Edge.Cuts) (width 0.15))
-  (segment (start 134.62 137.545) (end 134.62 133.33) (width 0.4) (layer F.Cu) (net 2))
-  (segment (start 133.3525 138.8125) (end 134.62 137.545) (width 0.4) (layer F.Cu) (net 2))
+  (gr_line (start 127 127) (end 133.35 127) (layer Edge.Cuts) (width 0.15))
   (segment (start 133.35 138.8125) (end 133.3525 138.8125) (width 0.4) (layer F.Cu) (net 2))
   (segment (start 143.775 141.915) (end 142.65 141.915) (width 0.4) (layer F.Cu) (net 2))
@@
   (segment (start 134.62 141.915) (end 136.75 141.915) (width 0.4) (layer F.Cu) (net 2))
   (segment (start 133.7325 138.8125) (end 134.62 139.7) (width 0.4) (layer F.Cu) (net 2))
-  (segment (start 138.850001 131.230001) (end 139.7 132.08) (width 0.4) (layer F.Cu) (net 4))
-  (segment (start 138.449999 130.829999) (end 138.850001 131.230001) (width 0.4) (layer F.Cu) (net 4))
-  (segment (start 133.449999 130.829999) (end 138.449999 130.829999) (width 0.4) (layer F.Cu) (net 4))
-  (segment (start 132.45 131.829998) (end 133.449999 130.829999) (width 0.4) (layer F.Cu) (net 4))
-  (segment (start 132.45 139.69) (end 132.45 131.829998) (width 0.4) (layer F.Cu) (net 4))
-  (segment (start 133.3475 140.5875) (end 132.45 139.69) (width 0.4) (layer F.Cu) (net 4))
-  (segment (start 133.35 140.5875) (end 133.3475 140.5875) (width 0.4) (layer F.Cu) (net 4))
-  (segment (start 148.075 132.08) (end 148.9725 132.08) (width 0.4) (layer F.Cu) (net 4))
-  (segment (start 145.535 129.54) (end 148.075 132.08) (width 0.4) (layer F.Cu) (net 4))
-  (segment (start 142.24 129.54) (end 145.535 129.54) (width 0.4) (layer F.Cu) (net 4))
-  (segment (start 139.7 132.08) (end 142.24 129.54) (width 0.4) (layer F.Cu) (net 4))
+  (segment (start 133.3525 138.8125) (end 134.62 137.545) (width 0.4) (layer F.Cu) (net 2))
+  (segment (start 134.62 137.545) (end 134.62 133.33) (width 0.4) (layer F.Cu) (net 2))
   (segment (start 148.9725 132.08) (end 148.9725 132.0775) (width 0.4) (layer F.Cu) (net 4))
-  (segment (start 139.7 132.08) (end 139.7 133.33) (width 0.4) (layer F.Cu) (net 4))
-  (segment (start 143.49 129.54) (end 139.7 133.33) (width 0.4) (layer F.Cu) (net 4))
-  (segment (start 151.13 129.54) (end 143.49 129.54) (width 0.4) (layer F.Cu) (net 4))
-  (segment (start 149.925002 137.16) (end 151.13 137.16) (width 0.4) (layer F.Cu) (net 4))
-  (segment (start 142.65 142.565) (end 144.520002 142.565) (width 0.4) (layer F.Cu) (net 4))
-  (segment (start 144.520002 142.565) (end 149.925002 137.16) (width 0.4) (layer F.Cu) (net 4))
-  (segment (start 151.13 137.16) (end 153.67 134.62) (width 0.4) (layer F.Cu) (net 4))
-  (segment (start 153.67 134.62) (end 153.67 132.08) (width 0.4) (layer F.Cu) (net 4))
-  (segment (start 153.67 132.08) (end 151.13 129.54) (width 0.4) (layer F.Cu) (net 4))
+  (segment (start 142.65 142.565) (end 144.455 142.565) (width 0.4) (layer F.Cu) (net 4))
   (segment (start 142.65 138.69) (end 142.65 139.315) (width 0.4) (layer F.Cu) (net 8))
   (segment (start 139.044003 134.580001) (end 142.65 138.185998) (width 0.4) (layer F.Cu) (net 8))
@@
   (segment (start 143.775001 134.865001) (end 143.775 139.965) (width 0.4) (layer F.Cu) (net 16))
   (segment (start 142.24 133.33) (end 143.775001 134.865001) (width 0.4) (layer F.Cu) (net 16))
-  (segment (start 131.28 143.51) (end 131.28 146.05) (width 0.4) (layer F.Cu) (net 17))
-  (segment (start 129.07 143.51) (end 131.28 143.51) (width 0.4) (layer F.Cu) (net 17))
-  (segment (start 134.045 143.865) (end 135.625 143.865) (width 0.4) (layer F.Cu) (net 18))
+  (segment (start 130.48 143.51) (end 130.48 149.86) (width 0.4) (layer F.Cu) (net 17))
+  (segment (start 128.27 143.51) (end 130.48 143.51) (width 0.4) (layer F.Cu) (net 17))
+  (segment (start 133.245 143.865) (end 135.625 143.865) (width 0.4) (layer F.Cu) (net 18))
   (segment (start 135.625 143.865) (end 136.75 143.865) (width 0.4) (layer F.Cu) (net 18))
-  (segment (start 133.69 143.51) (end 134.045 143.865) (width 0.4) (layer F.Cu) (net 18))
-  (segment (start 132.88 143.51) (end 133.69 143.51) (width 0.4) (layer F.Cu) (net 18))
+  (segment (start 132.89 143.51) (end 133.245 143.865) (width 0.4) (layer F.Cu) (net 18))
+  (segment (start 132.08 143.51) (end 132.89 143.51) (width 0.4) (layer F.Cu) (net 18))
   (segment (start 135.625 144.515) (end 136.75 144.515) (width 0.4) (layer F.Cu) (net 19))
-  (segment (start 133.515 144.515) (end 135.625 144.515) (width 0.4) (layer F.Cu) (net 19))
-  (segment (start 132.88 145.15) (end 133.515 144.515) (width 0.4) (layer F.Cu) (net 19))
-  (segment (start 132.88 146.05) (end 132.88 145.15) (width 0.4) (layer F.Cu) (net 19))
+  (segment (start 132.08 148.06) (end 135.625 144.515) (width 0.4) (layer F.Cu) (net 19))
+  (segment (start 132.08 149.86) (end 132.08 148.06) (width 0.4) (layer F.Cu) (net 19))
   (segment (start 146.52 145.96) (end 146.52 146.05) (width 0.4) (layer F.Cu) (net 20))
   (segment (start 145.075 144.515) (end 146.52 145.96) (width 0.4) (layer F.Cu) (net 20))
   (segment (start 142.65 144.515) (end 145.075 144.515) (width 0.4) (layer F.Cu) (net 20))
+  (segment (start 146.52 145.96) (end 146.52 149.86) (width 0.4) (layer F.Cu) (net 20))
   (segment (start 146.165 143.865) (end 146.52 143.51) (width 0.4) (layer F.Cu) (net 21))
   (segment (start 142.65 143.865) (end 146.165 143.865) (width 0.4) (layer F.Cu) (net 21))
   (segment (start 148.12 146.05) (end 148.12 143.51) (width 0.4) (layer F.Cu) (net 22))
   (segment (start 148.12 143.51) (end 150.33 143.51) (width 0.4) (layer F.Cu) (net 22))
+  (segment (start 148.12 146.05) (end 148.12 149.86) (width 0.4) (layer F.Cu) (net 22))
   (zone (net 4) (net_name GND) (layer F.Cu) (hatch edge 0.508)
     (connect_pads (clearance 0.508))
@@
     (polygon
       (pts
-        (xy 124.46 127) (xy 154.94 127) (xy 154.94 154.94) (xy 124.46 154.94)
+        (xy 124.46 129.54) (xy 127 127) (xy 154.94 127) (xy 154.94 154.94) (xy 124.46 154.94)
       )
     )
@@
     (polygon
       (pts
-        (xy 124.46 127) (xy 154.94 127) (xy 154.94 154.94) (xy 124.46 154.94)
+        (xy 124.46 129.54) (xy 127 127) (xy 154.94 127) (xy 154.94 154.94) (xy 124.46 154.94)
       )
     )

Commit message: Pin orientation
Parts:
- D1, D2, D3, D4: footprint LED_SMD:LED_0603_1608Metric -> LED_SMD:LED_0603_1608Metric_Pad0.82x1.00mm_HandSolder
- J1, J2: moved to B.Cu
- R1, R2: footprint Resistor_SMD:R_0603_1608Metric -> Resistor_SMD:R_0603_1608Metric_Pad0.99x1.00mm_HandSolder
- turned J1 to 270 degrees
- turned J2 to 270 degrees

Commit message: Moved LED node text
Changed lines of the file:
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@@
     )
   )
-  (gr_text "Pico\nNode\nLED" (at 125.73 133.35) (layer F.Cu)
+  (gr_text "Pico\nNode\nLED" (at 125.73 133.35) (layer F.Adhes)
     (effects (font (size 1.5 1.5) (thickness 0.3)) (justify left))
   )
@@
       )
     )
+  )
+  (zone (net 0) (net_name "") (layer F.Cu) (hatch edge 0.508)
+    (connect_pads (clearance 0.508))
+    (min_thickness 0.254)
+    (keepout (tracks not_allowed) (vias not_allowed) (copperpour allowed))
+    (fill (arc_segments 16) (thermal_gap 0.508) (thermal_bridge_width 0.508))
+    (polygon
+      (pts
+        (xy 130.175 137.16) (xy 130.175 134.62) (xy 131.445 134.62) (xy 131.445 129.54) (xy 125.73 129.54)
+        (xy 125.73 137.16)
+      )
+    )

Commit message: Discuss the node design
Connections:
- net Net-(J1-Pad2) renamed /SWCLK
- net Net-(J1-Pad4) renamed /SWDIO
- net Net-(J1-Pad5) renamed /nRST
- net Net-(J2-Pad1) renamed /Down
- net Net-(J2-Pad2) renamed /Left
- net Net-(J2-Pad3) renamed /Up
- net Net-(J2-Pad4) renamed /Right
