File: pcb/led-node/led-node.sch (KiCad schematic (older format))
At the start: 12 parts, among them J1 STM32_SWD, J2 PicoTalk, U1 STM32F030F4Px

Commit message: Pin orientation
Parts:
- D1, D2, D3, D4: footprint LED_SMD:LED_0603_1608Metric -> LED_SMD:LED_0603_1608Metric_Pad0.82x1.00mm_HandSolder
- R1, R2: footprint Resistor_SMD:R_0603_1608Metric -> Resistor_SMD:R_0603_1608Metric_Pad0.99x1.00mm_HandSolder
Changed lines of the file:
@@
 F 0 "D1" H 6642 2995 50  0000 C CNN
 F 1 "LED1" H 6642 3086 50  0000 C CNN
-F 2 "LED_SMD:LED_0603_1608Metric" H 6650 3250 50  0001 C CNN
+F 2 "LED_SMD:LED_0603_1608Metric_Pad0.82x1.00mm_HandSolder" H 6650 3250 50  0001 C CNN
 F 3 "" H 6650 3250 50  0001 C CNN
 	1    6650 3250
@@
 F 0 "D2" H 6642 3395 50  0000 C CNN
 F 1 "LED2" H 6642 3486 50  0000 C CNN
-F 2 "LED_SMD:LED_0603_1608Metric" H 6650 3650 50  0001 C CNN
+F 2 "LED_SMD:LED_0603_1608Metric_Pad0.82x1.00mm_HandSolder" H 6650 3650 50  0001 C CNN
 F 3 "" H 6650 3650 50  0001 C CNN
 	1    6650 3650
@@
 F 0 "D3" H 6642 3795 50  0000 C CNN
 F 1 "LED3" H 6642 3886 50  0000 C CNN
-F 2 "LED_SMD:LED_0603_1608Metric" H 6650 4050 50  0001 C CNN
+F 2 "LED_SMD:LED_0603_1608Metric_Pad0.82x1.00mm_HandSolder" H 6650 4050 50  0001 C CNN
 F 3 "" H 6650 4050 50  0001 C CNN
 	1    6650 4050
@@
 F 0 "D4" H 6642 4195 50  0000 C CNN
 F 1 "LED4" H 6642 4286 50  0000 C CNN
-F 2 "LED_SMD:LED_0603_1608Metric" H 6650 4450 50  0001 C CNN
+F 2 "LED_SMD:LED_0603_1608Metric_Pad0.82x1.00mm_HandSolder" H 6650 4450 50  0001 C CNN
 F 3 "" H 6650 4450 50  0001 C CNN
 	1    6650 4450
@@
 F 0 "R2" H 7220 4496 50  0000 L CNN
 F 1 "100" H 7220 4405 50  0000 L CNN
-F 2 "Resistor_SMD:R_0603_1608Metric" V 7080 4450 50  0001 C CNN
+F 2 "Resistor_SMD:R_0603_1608Metric_Pad0.99x1.00mm_HandSolder" V 7080 4450 50  0001 C CNN
 F 3 "" H 7150 4450 50  0001 C CNN
 	1    7150 4450
@@
 F 0 "R1" H 7220 3696 50  0000 L CNN
 F 1 "100" H 7220 3605 50  0000 L CNN
-F 2 "Resistor_SMD:R_0603_1608Metric" V 7080 3650 50  0001 C CNN
+F 2 "Resistor_SMD:R_0603_1608Metric_Pad0.99x1.00mm_HandSolder" V 7080 3650 50  0001 C CNN
 F 3 "" H 7150 3650 50  0001 C CNN
 	1    7150 3650

Commit message: Discuss the node design
Connections:
- net labels added: Down, Left, Right, SWCLK, SWDIO, Up, nRST
Changed lines of the file:
@@
 Wire Wire Line
 	6800 3650 7000 3650
+Text Label 3150 2900 0    50   ~ 0
+SWDIO
+Text Label 3150 3100 0    50   ~ 0
+SWCLK
+Text Label 3150 2800 0    50   ~ 0
+nRST
+Text Label 5150 3200 0    50   ~ 0
+Down
+Text Label 5150 2900 0    50   ~ 0
+Left
+Text Label 4050 3900 0    50   ~ 0
+Up
+Text Label 5150 3300 0    50   ~ 0
+Right
 $EndSCHEMATC
